File: single_board_controller.sch (EAGLE design)
At the start: 78 parts, among them IC1 MCP3008, IC2 MCP3008, K1 AQE12105, K2 AQE12105, P1 B9B-EH-A, P2 STEPPER, Q1 35A/25V/8.5mΩ, Q2 35A/25V/8.5mΩ, Q3 35A/25V/8.5mΩ, Q4 35A/25V/8.5mΩ, Q5 35A/25V/8.5mΩ, Q8 35A/25V/8.5mΩ, T1 BTA41, U1 OPTOISOLATOR-2SOIC8, U2 OPTOISOLATOR-2SOIC8, U3 OPTOISOLATOR-2SOIC8

Commit message: final pcb and schematic for Single board controller
Parts:
- R21: value 100 -> 100K
Connections:
- removed net +5V: K1.K, K2.K
- removed net VCC: U3.CL1, U3.CL2
- net 12V: now also K1.K, K2.K, U3.CL1, U3.CL2
- net OUT1N2: now also Q4.G; no longer Q5.G
- net OUT2N2: now also Q5.G; no longer Q4.G
Changed lines of the file:
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@@
 <part name="R19" library="SparkFun-Resistors" library_urn="urn:adsk.eagle:library:532" deviceset="0.3OHM" device="-0805-1/8W-1%" package3d_urn="urn:adsk.eagle:package:39651/1" value="2370"/>
 <part name="R20" library="SparkFun-Resistors" library_urn="urn:adsk.eagle:library:532" deviceset="0.3OHM" device="-0805-1/8W-1%" package3d_urn="urn:adsk.eagle:package:39651/1" value="30"/>
-<part name="R21" library="SparkFun-Resistors" library_urn="urn:adsk.eagle:library:532" deviceset="0.3OHM" device="-0805-1/8W-1%" package3d_urn="urn:adsk.eagle:package:39651/1" value="100"/>
+<part name="R21" library="SparkFun-Resistors" library_urn="urn:adsk.eagle:library:532" deviceset="0.3OHM" device="-0805-1/8W-1%" package3d_urn="urn:adsk.eagle:package:39651/1" value="100K"/>
 <part name="SUPPLY15" library="supply2" library_urn="urn:adsk.eagle:library:372" deviceset="GND" device=""/>
 <part name="SUPPLY16" library="SparkFun-PowerSymbols" library_urn="urn:adsk.eagle:library:530" deviceset="3.3V" device=""/>
@@
 <part name="GND3" library="SparkFun" deviceset="GND" device=""/>
 <part name="R6" library="SparkFun-Resistors" deviceset="10KOHM1/10W1%(0603)" device="0603" value="10K"/>
-<part name="P+14" library="supply1" library_urn="urn:adsk.eagle:library:371" deviceset="+5V" device=""/>
-<part name="P+15" library="supply1" library_urn="urn:adsk.eagle:library:371" deviceset="+5V" device=""/>
 <part name="HEATER2" library="con-jst-vh" deviceset="B2P-VH" device=""/>
 <part name="HEATER3" library="con-jst-vh" deviceset="B2P-VH" device=""/>
@@
 <part name="-12V_SUPPLY" library="con-jst-vh" deviceset="B2P-VH" device=""/>
 <part name="SUPPLY22" library="supply2" library_urn="urn:adsk.eagle:library:372" deviceset="GND" device=""/>
+<part name="P+11" library="SparkFun" deviceset="VCC" device="" value="HV"/>
+<part name="P+12" library="SparkFun" deviceset="VCC" device="" value="HV"/>
 </parts>
 <sheets>
@@
 <attribute name="VALUE" x="85.344" y="-2.032" size="1.778" layer="96" rot="MR90"/>
 </instance>
-<instance part="P+14" gate="1" x="40.64" y="0" smashed="yes" rot="MR0">
-<attribute name="VALUE" x="43.18" y="-5.08" size="1.778" layer="96" rot="MR90"/>
-</instance>
-<instance part="P+15" gate="1" x="40.64" y="-12.7" smashed="yes" rot="MR0">
-<attribute name="VALUE" x="43.18" y="-17.78" size="1.778" layer="96" rot="MR90"/>
-</instance>
 <instance part="HEATER2" gate="G$1" x="2.54" y="-5.08" smashed="yes" rot="R180">
 <attribute name="NAME" x="-3.81" y="1.905" size="1.778" layer="95" rot="R270"/>
@@
 <instance part="SUPPLY22" gate="GND" x="63.5" y="116.84" smashed="yes" rot="MR0">
 <attribute name="VALUE" x="65.405" y="113.665" size="1.778" layer="96" rot="MR0"/>
+</instance>
+<instance part="P+11" gate="1" x="45.72" y="-5.08" smashed="yes" rot="MR0">
+<attribute name="VALUE" x="46.736" y="-1.524" size="1.778" layer="96" rot="MR0"/>
+</instance>
+<instance part="P+12" gate="1" x="43.18" y="-17.78" smashed="yes" rot="MR0">
+<attribute name="VALUE" x="44.196" y="-14.224" size="1.778" layer="96" rot="MR0"/>
 </instance>
 </instances>
@@
 <junction x="-5.08" y="50.8"/>
 </segment>
+<segment>
+<pinref part="K1" gate="A" pin="K"/>
+<wire x1="40.64" y1="-5.08" x2="45.72" y2="-5.08" width="0.1524" layer="91"/>
+<pinref part="P+11" gate="1" pin="VCC"/>
+<label x="45.72" y="-5.08" size="1.778" layer="95"/>
+</segment>
+<segment>
+<pinref part="P+10" gate="1" pin="VCC"/>
+<pinref part="U3" gate="G$1" pin="CL1"/>
+<wire x1="93.98" y1="-15.24" x2="91.44" y2="-15.24" width="0.1524" layer="91"/>
+<junction x="93.98" y="-15.24"/>
+<wire x1="91.44" y1="-15.24" x2="91.44" y2="-20.32" width="0.1524" layer="91"/>
+<pinref part="U3" gate="G$1" pin="CL2"/>
+<wire x1="91.44" y1="-20.32" x2="93.98" y2="-20.32" width="0.1524" layer="91"/>
+</segment>
+<segment>
+<wire x1="40.64" y1="-17.78" x2="43.18" y2="-17.78" width="0.1524" layer="91"/>
+<pinref part="P+12" gate="1" pin="VCC"/>
+<label x="43.18" y="-17.78" size="1.778" layer="95"/>
+<pinref part="K2" gate="A" pin="K"/>
+</segment>
 </net>
 <net name="N$3" class="0">
@@
 <wire x1="137.16" y1="139.7" x2="180.34" y2="139.7" width="0.1524" layer="91"/>
 <junction x="180.34" y="139.7"/>
-</segment>
-</net>
-<net name="+5V" class="0">
-<segment>
-<pinref part="P+14" gate="1" pin="+5V"/>
-<wire x1="40.64" y1="-2.54" x2="40.64" y2="-5.08" width="0.1524" layer="91"/>
-<pinref part="K1" gate="A" pin="K"/>
-</segment>
-<segment>
-<pinref part="P+15" gate="1" pin="+5V"/>
-<wire x1="40.64" y1="-15.24" x2="40.64" y2="-17.78" width="0.1524" layer="91"/>
-<pinref part="K2" gate="A" pin="K"/>
 </segment>
 </net>
@@
 <net name="OUT2N2" class="0">
 <segment>
-<wire x1="83.82" y1="-7.62" x2="83.82" y2="-22.86" width="0.1524" layer="91"/>
-<wire x1="83.82" y1="-22.86" x2="83.82" y2="-30.48" width="0.1524" layer="91"/>
-<wire x1="83.82" y1="-30.48" x2="73.66" y2="-30.48" width="0.1524" layer="91"/>
+<wire x1="83.82" y1="-7.62" x2="83.82" y2="-17.78" width="0.1524" layer="91"/>
 <pinref part="R6" gate="G$1" pin="1"/>
-<pinref part="Q4" gate="NMOS" pin="G"/>
 <pinref part="U3" gate="G$1" pin="EM2"/>
+<wire x1="83.82" y1="-17.78" x2="83.82" y2="-22.86" width="0.1524" layer="91"/>
 <wire x1="93.98" y1="-22.86" x2="83.82" y2="-22.86" width="0.1524" layer="91"/>
-<junction x="83.82" y="-22.86"/>
+<pinref part="Q5" gate="NMOS" pin="G"/>
+<wire x1="63.5" y1="-17.78" x2="83.82" y2="-17.78" width="0.1524" layer="91"/>
+<junction x="83.82" y="-17.78"/>
 </segment>
 </net>
@@
 <segment>
 <wire x1="88.9" y1="-7.62" x2="88.9" y2="-17.78" width="0.1524" layer="91"/>
-<wire x1="88.9" y1="-17.78" x2="63.5" y2="-17.78" width="0.1524" layer="91"/>
 <pinref part="R5" gate="G$1" pin="1"/>
-<pinref part="Q5" gate="NMOS" pin="G"/>
 <pinref part="U3" gate="G$1" pin="EM1"/>
 <wire x1="93.98" y1="-17.78" x2="88.9" y2="-17.78" width="0.1524" layer="91"/>
+<wire x1="88.9" y1="-30.48" x2="73.66" y2="-30.48" width="0.1524" layer="91"/>
+<pinref part="Q4" gate="NMOS" pin="G"/>
+<wire x1="88.9" y1="-17.78" x2="88.9" y2="-30.48" width="0.1524" layer="91"/>
 <junction x="88.9" y="-17.78"/>
 </segment>
@@
 </segment>
 </net>
-<net name="VCC" class="0">
-<segment>
-<pinref part="P+10" gate="1" pin="VCC"/>
-<pinref part="U3" gate="G$1" pin="CL1"/>
-<wire x1="93.98" y1="-15.24" x2="91.44" y2="-15.24" width="0.1524" layer="91"/>
-<junction x="93.98" y="-15.24"/>
-<wire x1="91.44" y1="-15.24" x2="91.44" y2="-20.32" width="0.1524" layer="91"/>
-<pinref part="U3" gate="G$1" pin="CL2"/>
-<wire x1="91.44" y1="-20.32" x2="93.98" y2="-20.32" width="0.1524" layer="91"/>
-</segment>
-</net>
